Commit message: Finished description and added rviz2 launch script

File: description/robot_core.xacro (robot description, xacro)
@@ -1,4 +1,5 @@
 <?xml version="1.0"?>
 <robot xmlns:xacro="http://www.ros.org/wiki/xacro">
+    <xacro:include filename="inertial_macros.xacro" />
     <!-- Materials -->
         <material name="black">
@@ -11,5 +12,5 @@
         <link name="base_link">
             <visual>
-                <origin xyz="0 0 0.05"/>
+                <origin xyz="0 0 0.025"/>
                 <geometry>
                     <box size="0.05 0.05 0.05"/>
@@ -17,20 +18,38 @@
                 <material name="white"/>
             </visual>
+            <collision>
+                <origin xyz="0 0 0.025"/>
+                <geometry>
+                    <box size="0.05 0.05 0.05"/>
+                </geometry>
+            </collision>
+            <xacro:inertial_box mass="0.1" x="0.05" y="0.05" z="0.05">
+                <origin xyz="0 0 0.025" rpy="0.0 0.0 0.0"/>
+            </xacro:inertial_box>
         </link>
         <joint name="arm_joint" type="revolute">
-            <origin xyz="0 0 0.1"/>
+            <origin xyz="0 0 0.05"/>
             <parent link="base_link"/>
             <child link="arm_link"/>
             <axis xyz="0 0 1"/>
-            <limit lower="-${pi/2}" upper="${pi/2}" effort="100" velocity="10"/>
+            <limit lower="0" upper="${pi}" effort="100" velocity="10"/>
         </joint>
         <link name="arm_link">
             <visual>
-                <origin xyz="0 0 0.05"/>
+                <origin xyz="0.05 0 0"/>
                 <geometry>
-                    <box size="0.05 0.05 0.1"/>
+                    <box size="0.1 0.02 0.01"/>
                 </geometry>
                 <material name="black"/>
             </visual>
+            <collision>
+                <origin xyz="0.05 0 0"/>
+                <geometry>
+                    <box size="0.1 0.02 0.01"/>
+                </geometry>
+            </collision>
+            <xacro:inertial_box mass="0.1" x="0.1" y="0.02" z="0.01">
+                <origin xyz="0.05 0 0" rpy="0.0 0.0 0.0"/>
+            </xacro:inertial_box>
         </link>
 </robot>
